File: src/sensor_pcb/_autosave-sensor_pcb.kicad_sch (KiCad schematic)
At the start: 15 parts, among them Q1 NPN BJT 40V 200mA, U1 SHT45-AD1B, U2 16-bit ADC

Commit message: pressure sensor added
Parts:
- added C3, C4: 100nF, Capacitor_SMD:C_0201_0603Metric, symbol #dzdb:g_cap/C-100n-0201
- added R10, R11: 100k, Resistor_SMD:R_0603_1608Metric, symbol #dzdb:g_res/R-100k-0603
- added U4: BMP581, dz_sens:BMP581, symbol #dzdb:s_sens/D-BOSCH-BMP581
Connections:
- net GND: now also C3.2, C4.2, R11.2, U4.3 (VSS_1), U4.8 (VSS_2), U4.9 (VSS_3)
- net SCL: now also U4.2 (SCK)
- net SDA: now also U4.4 (SDI)
- net VDD: now also C3.1, C4.1, U4.1 (VDDIO), U4.10 (VDD)
- net at U2.4 (AIN0): now also R10.2, R11.1
- new net sensor: R10.1
Other:
- added sheet stm (untitled.kicad_sch)
- note added: "Add resistors in series to grab 5v to 3.3 from connector for sensor"
- note added: "Humidity + Temp."
- note added: "change resistors to loose less e"
- note removed: "Pressure + Temp."
- moved on the sheet: C2, R7, R8, R9, U2
