File: src/sensor_pcb/stm.kicad_sch (KiCad schematic)
At the start: 1 part, among them U3 STM32L451CET6

Commit message: 8 pin connectors added
Connections:
- net ls 1: now reaches U3.18 (PB0)
- net ls 2: now reaches U3.19 (PB1)
Changed lines of the file:
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@@
 	(generator_version "9.0")
 	(paper "A4")
+	(wire
+		(pts
+			(xy 48.26 91.44) (xy 54.61 91.44)
+		)
+		(stroke
+			(width 0)
+			(type default)
+		)
+	)
+	(wire
+		(pts
+			(xy 48.26 93.98) (xy 54.61 93.98)
+		)
+		(stroke
+			(width 0)
+			(type default)
+		)
+	)
+	(wire
+		(pts
+			(xy 48.26 88.9) (xy 54.61 88.9)
+		)
+		(stroke
+			(width 0)
+			(type default)
+		)
+	)
+	(wire
+		(pts
+			(xy 48.26 96.52) (xy 54.61 96.52)
+		)
+		(stroke
+			(width 0)
+			(type default)
+		)
+	)
+	(wire
+		(pts
+			(xy 48.26 101.6) (xy 54.61 101.6)
+		)
+		(stroke
+			(width 0)
+			(type default)
+		)
+	)
+	(wire
+		(pts
+			(xy 48.26 99.06) (xy 54.61 99.06)
+		)
+		(stroke
+			(width 0)
+			(type default)
+		)
+	)
+	(wire
+		(pts
+			(xy 48.26 104.14) (xy 54.61 104.14)
+		)
+		(stroke
+			(width 0)
+			(type default)
+		)
+	)
+	(wire
+		(pts
+			(xy 48.26 86.36) (xy 54.61 86.36)
+		)
+		(stroke
+			(width 0)
+			(type default)
+		)
+	)
+	(hierarchical_label "ls 2"
+		(shape input)
+		(at 48.26 88.9 180)
+		(effects
+			(font
+				(size 1.27 1.27)
+			)
+			(justify right)
+		)
+	)
+	(hierarchical_label "ls 1"
+		(shape input)
+		(at 48.26 86.36 180)
+		(effects
+			(font
+				(size 1.27 1.27)
+			)
+			(justify right)
+		)
+	)
 	(symbol
 		(lib_id "#dzdb:s_mcu/M-STM-STM32L451CET6")

Commit message: v1 complete
Connections:
- net PA0: now reaches U3.10 (PA0)
- net PA1: now reaches U3.11 (PA1)
- net PA2: now reaches U3.12 (PA2)
- net PA3: now reaches U3.13 (PA3)
- net PA4: now reaches U3.14 (PA4)
- net PA5: now reaches U3.15 (PA5)
- net GND: now reaches U3.23 (VSS), U3.35 (VSS), U3.47 (VSS)
- net GND: now also U3.8 (VSSA)
- net VDD: now reaches U3.24 (VDD)
- net ls 1 renamed PB0
- net ls 2 renamed PB1
Other:
- company: (none) -> Giacomo Raggi
- title: (none) -> Sensor_pcb: stm
Changed lines of the file:
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@@
 	(generator_version "9.0")
 	(paper "A4")
+	(title_block
+		(title "Sensor_pcb: stm")
+		(date "2025-10-21")
+		(company "Giacomo Raggi")
+	)
+	(junction
+		(at 72.39 132.08)
+		(diameter 0)
+		(color 0 0 0 0)
+	)
 	(wire
 		(pts
@@
 	(wire
 		(pts
+			(xy 72.39 140.97) (xy 71.12 140.97)
+		)
+		(stroke
+			(width 0)
+			(type default)
+		)
+	)
+	(wire
+		(pts
+			(xy 72.39 132.08) (xy 72.39 140.97)
+		)
+		(stroke
+			(width 0)
+			(type default)
+		)
+	)
+	(wire
+		(pts
 			(xy 48.26 96.52) (xy 54.61 96.52)
 		)
@@
 	(wire
 		(pts
+			(xy 69.85 132.08) (xy 72.39 132.08)
+		)
+		(stroke
+			(width 0)
+			(type default)
+		)
+	)
+	(wire
+		(pts
 			(xy 48.26 99.06) (xy 54.61 99.06)
 		)
@@
 		)
 	)
-	(hierarchical_label "ls 2"
+	(hierarchical_label "PB1"
 		(shape input)
 		(at 48.26 88.9 180)
@@
 		)
 	)
-	(hierarchical_label "ls 1"
+	(hierarchical_label "PA2"
+		(shape input)
+		(at 85.09 66.04 0)
+		(effects
+			(font
+				(size 1.27 1.27)
+			)
+			(justify left)
+		)
+	)
+	(hierarchical_label "PA4"
+		(shape input)
+		(at 85.09 71.12 0)
+		(effects
+			(font
+				(size 1.27 1.27)
+			)
+			(justify left)
+		)
+	)
+	(hierarchical_label "PB0"
 		(shape input)
 		(at 48.26 86.36 180)
@@
 		)
 	)
+	(hierarchical_label "PA5"
+		(shape input)
+		(at 85.09 73.66 0)
+		(effects
+			(font
+				(size 1.27 1.27)
+			)
+			(justify left)
+		)
+	)
+	(hierarchical_label "GND"
+		(shape input)
+		(at 71.12 140.97 180)
+		(effects
+			(font
+				(size 1.27 1.27)
+			)
+			(justify right)
+		)
+	)
+	(hierarchical_label "PA3"
+		(shape input)
+		(at 85.09 68.58 0)
+		(effects
+			(font
+				(size 1.27 1.27)
+			)
+			(justify left)
+		)
+	)
+	(hierarchical_label "VDD"
+		(shape input)
+		(at 67.31 53.34 90)
+		(effects
+			(font
+				(size 1.27 1.27)
+			)
+			(justify left)
+		)
+	)
+	(hierarchical_label "PA0"
+		(shape input)
+		(at 85.09 60.96 0)
+		(effects
+			(font
+				(size 1.27 1.27)
+			)
+			(justify left)
+		)
+	)
+	(hierarchical_label "PA1"
+		(shape input)
+		(at 85.09 63.5 0)
+		(effects
+			(font
+				(size 1.27 1.27)
+			)
+			(justify left)
+		)
+	)

Commit message: schematic update
Connections:
- net PA6: now reaches U3.16 (PA6)
- net PA9: now reaches U3.30 (PA9)
Changed lines of the file:
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@@
+		)
+	)
+	(hierarchical_label "PA9"
+		(shape input)
+		(at 85.09 83.82 0)
+		(effects
+			(font
+				(size 1.27 1.27)
+			)
+			(justify left)
 		)
 	)
@@
 		)
 	)
+	(hierarchical_label "PA6"
+		(shape input)
+		(at 85.09 76.2 0)
+		(effects
+			(font
+				(size 1.27 1.27)
+			)
+			(justify left)
+		)
+	)

Commit message: intermediate changes
Connections:
- net PB2: now reaches U3.20 (PB2)
- net PB13: now reaches U3.26 (PB13)
- net PB3: now reaches U3.39 (PB3)
- net PB4: now reaches U3.40 (PB4)
- net PB5: now reaches U3.41 (PB5)
- net PB6: now reaches U3.42 (PB6)
- net PB7: now reaches U3.43 (PB7)
Changed lines of the file:
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@@
+	(wire
+		(pts
+			(xy 48.26 119.38) (xy 54.61 119.38)
+		)
+		(stroke
+			(width 0)
+			(type default)
+		)
+	)
 	(wire
 		(pts
@@
 		)
 	)
+	(hierarchical_label "PB3"
+		(shape input)
+		(at 48.26 93.98 180)
+		(effects
+			(font
+				(size 1.27 1.27)
+			)
+			(justify right)
+		)
+	)
 	(hierarchical_label "PB1"
 		(shape input)
@@
 		)
 	)
+	(hierarchical_label "PB6"
+		(shape input)
+		(at 48.26 101.6 180)
+		(effects
+			(font
+				(size 1.27 1.27)
+			)
+			(justify right)
+		)
+	)
 	(hierarchical_label "PA2"
 		(shape input)
@@
 		)
 	)
+	(hierarchical_label "PB2"
+		(shape input)
+		(at 48.26 91.44 180)
+		(effects
+			(font
+				(size 1.27 1.27)
+			)
+			(justify right)
+		)
+	)
+	(hierarchical_label "PB5"
+		(shape input)
+		(at 48.26 99.06 180)
+		(effects
+			(font
+				(size 1.27 1.27)
+			)
+			(justify right)
+		)
+	)
+	(hierarchical_label "PB4"
+		(shape input)
+		(at 48.26 96.52 180)
+		(effects
+			(font
+				(size 1.27 1.27)
+			)
+			(justify right)
+		)
+	)
 	(hierarchical_label "GND"
 		(shape input)
@@
 		)
 	)
+	(hierarchical_label "PB13"
+		(shape input)
+		(at 48.26 119.38 180)
+		(effects
+			(font
+				(size 1.27 1.27)
+			)
+			(justify right)
+		)
+	)
 	(hierarchical_label "VDD"
 		(shape input)
@@
 		)
 	)
+	(hierarchical_label "PB7"
+		(shape input)
+		(at 48.26 104.14 180)
+		(effects
+			(font
+				(size 1.27 1.27)
+			)
+			(justify right)
+		)
+	)
