File: src/sensor_pcb/_autosave-sensor_stm.kicad_sch (KiCad schematic)
At the start: 16 parts, among them J6 FTSH-107-02-L-DV, SW1 Button Switch SPST-No, U3 STM32L451CET6, Y1 16.0MHz

Commit message: clearing up errors
Connections:
- net nRST: now also C8.1, R1.2, SW1.2, U3.7 (NRST)
- no-connect marks 21 -> 29
Other:
- note added: "Crystall"
- note added: "Decoupling"
- note added: "STM"
- note removed: "CRYSTALL"
- note removed: "STM SCHEMATIC"
- moved on the sheet: C26, C31, J6, Y1
