File: src/sensor_pcb/sensor_stm.kicad_sch (KiCad schematic)
At the start: 16 parts, among them J6 FTSH-107-02-L-DV, SW1 Button Switch SPST-No, U3 STM32L451CET6, Y1 16.0MHz

Commit message: final changes before review
Parts:
- removed C12: 4.7uF, Capacitor_SMD:C_0402_1005Metric, symbol #dzdb:g_cap/C-4.7u-0402
- removed R40: 0, Resistor_SMD:R_0201_0603Metric, symbol #dzdb:g_res/R-0-0201
- added C13, C14: 100nF, Capacitor_SMD:C_0603_1608Metric, symbol #dzdb:g_cap/C-100n-0603
- added C15: 4.7nF, Capacitor_SMD:C_0603_1608Metric, symbol #dzdb:g_cap/C-4.7n-0603
- added R41: 0, Resistor_SMD:R_0603_1608Metric, symbol #dzdb:g_res/R-0-0603
Connections:
- net +3.3V: now also C13.1, C14.1, C15.1, R41.1, R41.2
- net GND: now also C13.2, C14.2, C15.2
- net nRST: now also C8.1, R1.2, SW1.2, U3.7 (NRST)
- no-connect marks 21 -> 29
Other:
- note added: "Crystall"
- note added: "Decoupling"
- note added: "STM"
- note removed: "CRYSTALL"
- note removed: "STM SCHEMATIC"
- moved on the sheet: C26, C31, J6, Y1
