File: src/sensor_pcb/sensor_stm.kicad_sch (KiCad schematic)
At the start: 18 parts, among them J6 FTSH-107-02-L-DV, SW1 Button Switch SPST-No, U3 STM32L451CET6, Y1 16.0MHz

Commit message: bom process
Parts:
- added D21, D22: 710-82402374, Package_TO_SOT_SMD:SOT-23-5, symbol #dzdb:s_dio/WURT-710-82402374
Connections:
- net GND: now also D21.2 (A), D22.2 (A)
- net JTAG_TCK/SWCLK: now also D21.4 (K)
- net JTAG_TDI: now also D21.1 (K)
- net JTAG_TDO/SWD: now also D21.3 (K)
- net JTAG_TMS/SWDIO: now also D21.5 (K)
- net UART0.RX: now also D22.3 (K)
- net UART0.TX: now also D22.4 (K)
- net nRST: now also D22.5 (K)
- no-connect marks 29 -> 30
Other:
- title: (none) -> Sensor PCB: stm

Commit message: changed to bigger footprints on resistors
Parts:
- FB2: SPN 81-BLM18SP101SN1 -> 81-BLM18SP101SN1D
- R41: SPN 594-RCA06030000ZSTA -> 71-RCA06030000ZSTA
Changed lines of the file:
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@@
 			)
 		)
-		(property "SPN" "594-RCA06030000ZSTA"
+		(property "SPN" "71-RCA06030000ZSTA"
 			(at 193.04 31.75 0)
 			(effects
@@
 			)
 		)
-		(property "SPN" "81-BLM18SP101SN1"
+		(property "SPN" "81-BLM18SP101SN1D"
 			(at 193.04 44.45 0)
 			(effects
