File: src/sensor_pcb/sensor_pcb.kicad_pcb (KiCad board)
At the start: 4 copper layers, 64 x 58.4 mm, 93 parts, among them IC1 TCAN3414DRBR, J1 66200421024, J2 643280100305, J3 66200821024, J4 643280100305, J5 66200821024, J6 FTSH-107-02-L-DV, J7 66200421024, Q1 NPN BJT 40V 200mA, Q2 NPN BJT 40V 200mA, Q3 NPN BJT 40V 200mA, Q4 NPN BJT 40V 200mA, Q5 NPN BJT 40V 200mA, Q6 NPN BJT 40V 200mA, Q7 NPN BJT 40V 200mA, Q8 NPN BJT 40V 200mA, SW1 Button Switch SPST-No, U1 SHT45-AD1B, U2 16-bit ADC, U3 STM32L451CET6, U4 BMP581, Y1 16.0MHz

Commit message: quick save on progress
Parts:
- removed R18, R23, R27, R31, R35, R39: 240, Resistor_SMD:R_0603_1608Metric
- added D16: 710-82402374, Package_TO_SOT_SMD:SOT-23-5, F.Cu at (151.1, 74.1)
- added D17: 710-82402374, Package_TO_SOT_SMD:SOT-23-5, F.Cu at (151.8, 88.9)
- added D18: SMBJ3.3A, Diode_SMD:D_SMB, F.Cu at (161.8, 70.2)
- added D19: SMBJ3.3A, Diode_SMD:D_SMB, F.Cu at (179.2, 70.3)
- added D20: SMBJ3.3A, Diode_SMD:D_SMB, F.Cu at (171.7, 70.4)
- added D21: 710-82402374, Package_TO_SOT_SMD:SOT-23-5, F.Cu at (184.4, 89.7)
- added D22: 710-82402374, Package_TO_SOT_SMD:SOT-23-5, F.Cu at (169.1, 98.3)
- added D5: 710-82402374, Package_TO_SOT_SMD:SOT-23-5, F.Cu at (186.2, 78.2)
- added LED1: 710-150060RS83000, dz_dio:Wuerth_LED_150060RS83000, F.Cu at (201.7, 61.1)
- added R40: 100, Resistor_SMD:R_0402_1005Metric, F.Cu at (189.8, 72.3)
- added R42: 1k, Resistor_SMD:R_0603_1608Metric, F.Cu at (199.7, 61.2)
- added R43: 1k, Resistor_SMD:R_0603_1608Metric, F.Cu at (187.5, 92.1)
- added R44: 1k, Resistor_SMD:R_0603_1608Metric, F.Cu at (149.9, 103.8)
- added R45: 1k, Resistor_SMD:R_0603_1608Metric, F.Cu at (149.9, 110.0)
- added R46: 1k, Resistor_SMD:R_0603_1608Metric, F.Cu at (150.0, 98.4)
- added R47: 1k, Resistor_SMD:R_0603_1608Metric, F.Cu at (187.8, 107.0)
- added R48: 1k, Resistor_SMD:R_0603_1608Metric, F.Cu at (188.1, 97.1)
- added TP1: Test Point, TestPoint:TestPoint_Pad_D1.5mm, F.Cu at (137.1, 56.4)
- added TP2: Test Point, TestPoint:TestPoint_Pad_D1.5mm, F.Cu at (137.1, 59.6)
- added TP3: Test Point, TestPoint:TestPoint_Pad_D1.5mm, F.Cu at (137.2, 62.4)
- added TP4: Test Point, TestPoint:TestPoint_Pad_D1.5mm, F.Cu at (137.2, 65.8)
- added TP5: Test Point, TestPoint:TestPoint_Pad_D1.5mm, F.Cu at (161.2, 80.5)
- added TP6: Test Point, TestPoint:TestPoint_Pad_D1.5mm, F.Cu at (158.4, 80.5)
- added Z1: 824094024, dz_dio:SOT95P240X104-3N, F.Cu at (200.9, 64.6)
- added Z2: 824094024, dz_dio:SOT95P240X104-3N, F.Cu at (138.3, 69.9)
- D9: value 150060RS73220 -> 710-82402374; footprint dz_dio:LED_0603 -> Package_TO_SOT_SMD:SOT-23-5
- R14, R19: value 240 -> 1k
- moved D9 44.5 mm to (188.9, 88.5), turned to 180 degrees
- moved R19 38.8 mm to (150.1, 94.0), turned to 0 degrees
- moved R14 10.1 mm to (188.0, 102.1)
- moved D6 2.50 mm to (185.2, 70.2), turned to -90 degrees
- moved D4 1.77 mm to (143.9, 69.3)
- moved D15 0.14 mm to (152.1, 109.1)
- moved R33 0.08 mm to (141.8, 104.0)
Connections:
- D1 pad A: Net-(D7-A1) -> Net-(D1-PadA)
- D1 pad C: +3.3V -> GND
- D7 pad 1: Net-(D7-A1) -> +3.3V
- R14 pad 1: /s 1.1 -> /s 3.1
- R14 pad 2: Net-(D2-PadA) -> Net-(D10-PadA)
- R19 pad 1: /s 3.1 -> /s 5.1
- R19 pad 2: Net-(D10-PadA) -> Net-(D11-PadA)
- R2 pad 2: Net-(D7-A1) -> +3.3V
Routing:
- net GND: track 39.6 -> 86.7 mm, vias 21 -> 42
- net /CAN_L: track 76.6 -> 110.6 mm, vias 1 -> 4
- net /CAN_H: track 73.0 -> 101.7 mm
- net +5V: track 7.76 -> 35.2 mm
- net +3.3V: track 90.2 -> 112.3 mm
- net /sensor_stm/JTAG_TCK/SWCLK: track 15.1 -> 37.1 mm, vias 2 -> 3
- net /ls 3.1: track 35.2 -> 50.4 mm, vias 1 -> 2
- net /sensor_stm/JTAG_TMS/SWDIO: track 11.6 -> 26.2 mm, vias 2 -> 4
- net /ls 7.1: track 22.8 -> 37.2 mm
- net /ls 6.1: track 25.1 -> 38.9 mm, vias 2 -> 3
- net /ls 1.1: track 26.6 -> 36.9 mm
- net /sensor_stm/SDA: track 54.4 -> 64.2 mm
- net /sensor_stm/SCL: track 49.9 -> 59.0 mm, vias 2 -> 4
- net /sensor_stm/JTAG_TDO/SWD: track 17.5 -> 26.6 mm, vias 2 -> 4
- net /sensor_stm/JTAG_TDI: track 21.7 -> 30.5 mm, vias 2 -> 4
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Other:
- board size 64 x 58.4 mm -> 67.6 x 56.9 mm
