File: src/sensor_pcb/sensor_pcb.kicad_pcb (KiCad board)
At the start: 4 copper layers, 67.6 x 56.9 mm, 112 parts, among them IC1 TCAN3414DRBR, J1 66200421024, J2 643280100305, J3 66200821024, J4 643280100305, J5 66200821024, J6 FTSH-107-02-L-DV, J7 66200421024, Q1 NPN BJT 40V 200mA, Q2 NPN BJT 40V 200mA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

Commit message: changes from wrong db
Parts:
- removed C5: 100nF, Capacitor_SMD:C_0402_1005Metric
- added C12: 100nF, Capacitor_SMD:C_0603_1608Metric, F.Cu at (166.3, 75.5)
- added G***: LOGO, dz_art:giacomo_logo, B.Cu at (185.6, 107.3)
- C1, C3, C4: footprint Capacitor_SMD:C_0201_0603Metric -> Capacitor_SMD:C_0603_1608Metric
- C2: footprint Capacitor_SMD:C_0402_1005Metric -> Capacitor_SMD:C_0603_1608Metric
- moved C4 18.8 mm to (180.4, 89.1)
- moved C3 3.75 mm to (172.2, 75.2), turned to -90 degrees
- moved IC1 1.41 mm to (179.4, 85.4)
- moved C1 0.57 mm to (159.6, 73.6)
- moved C2 0.56 mm to (183.7, 80.7)
Routing:
- net /CAN_L: track 110.6 -> 105.2 mm
- net +3.3V: track 112.3 -> 115.9 mm, vias 37 -> 36
- net GND: track 86.7 -> 83.5 mm, vias 42 -> 134
- net /CAN_H: track 101.7 -> 103.1 mm
- net /sensor_stm/CAN.RX: track 13.2 -> 14.5 mm
- net /sensor_stm/JTAG_TDO/SWD: track 26.6 -> 27.9 mm
- net /sensor_stm/CAN.TX: track 8.89 -> 9.89 mm
- added copper zone on B.Cu, net GND
Other:
- board text added: "Nautilus Sensor PCB v1 (9/12/25)"
- board text added: "creato da Focss"

Commit message: symbol update for spn
Parts:
- removed R40: 100, Resistor_SMD:R_0402_1005Metric
- added R3: 100, Resistor_SMD:R_0603_1608Metric, F.Cu at (189.1, 68.9)
- R2: footprint Resistor_SMD:R_0402_1005Metric -> Resistor_SMD:R_0603_1608Metric
- moved R2 3.52 mm to (189.6, 72.5), turned to 180 degrees
Connections:
- R2 pad 1: Net-(J2-Pin_3) -> +3.3V
- R2 pad 2: +3.3V -> Net-(D1-PadA)
Routing:
- net Net-(J2-Pin_3): track 11.2 -> 10.4 mm
