File: src/sensor_pcb/_autosave-sensor_pcb.kicad_pcb (KiCad board)
At the start: 4 copper layers, 67.6 x 56.9 mm, 112 parts, among them IC1 TCAN3414DRBR, J1 66200421024, J2 643280100305, J3 66200821024, J4 643280100305, J5 66200821024, J6 FTSH-107-02-L-DV, J7 66200421024, Q1 NPN BJT 40V 200mA, Q2 NPN BJT 40V 200mA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

Commit message: bom process
Parts:
- added G***: LOGO, dz_art:giacomo_logo, B.Cu at (185.6, 107.3)
Other:
- board text added: "Nautilus Sensor PCB v1 (9/12/25)"
- board text added: "creato da Focss"
